File: swallow/kicad/swallow/swallow.kicad_pcb (KiCad board)
At the start: 2 copper layers, 75.8 x 74.2 mm, 36 parts, among them J1 Raspberry Pi 3/4 B, J10 evens, J2 echo2, J3 ground, J4 VCC, J5 echo3, J6 echo4, J7 echo1, J8 power terminal, J9 odds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

Commit message: swallow PCB update - kamangir/bolt#746
Connections:
- C1 pad 2: Net-(D1-K) -> GND
- D1 pad 1: Net-(D1-K) -> GND
- D2 pad 1: Net-(D1-K) -> GND
- D3 pad 1: Net-(D1-K) -> GND
- D4 pad 2: Net-(D1-K) -> GND
- D5 pad 1: Net-(D1-K) -> GND
- D6 pad 1: Net-(D1-K) -> GND
- D7 pad 1: Net-(D1-K) -> GND
- D8 pad 1: Net-(D1-K) -> GND
- J1 pad 25: Net-(D1-K) -> GND
- J1 pad 6: Net-(D1-K) -> GND
- J10 pad 3: Net-(D1-K) -> GND
- J3 pad 1: Net-(D1-K) -> GND
- J3 pad 2: Net-(D1-K) -> GND
- J3 pad 3: Net-(D1-K) -> GND
- J3 pad 4: Net-(D1-K) -> GND
- J3 pad 5: Net-(D1-K) -> GND
- J3 pad 6: Net-(D1-K) -> GND
- J3 pad 7: Net-(D1-K) -> GND
- J3 pad 8: Net-(D1-K) -> GND
- J8 pad 1: Net-(D1-K) -> GND
- J9 pad 13: Net-(D1-K) -> GND
- R10 pad 2: Net-(D1-K) -> GND
- R13 pad 2: Net-(D1-K) -> GND
- R5 pad 2: Net-(D1-K) -> GND
- R7 pad 2: Net-(D1-K) -> GND
- SW1 pad 1: Net-(D1-K) -> GND
Routing:
- net GND: track 0.00 -> 276.1 mm
- net Net-(D1-K): track 244.2 -> 0.00 mm
- added copper zone on F.Cu, net GND
Other:
- board text added: "swallow - v10 Karband / Kamangir"
- board text removed: "swallow - v9 Karband / Kamangir"
