File: swallow/kicad/swallow/swallow.kicad_sch (KiCad schematic)
At the start: 35 parts, among them J1 Raspberry_Pi_2_3, J10 evens, J2 echo2, J3 ground, J4 VCC, J5 echo3, J6 echo4, J7 echo1, J8 power terminal, J9 odds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

Commit message: ++
Changed lines of the file:
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@@
 		)
 	)
-	(label "v16"
+	(label "v17"
 		(at 267.97 194.31 0)
 		(effects
